File: Eagle/s3-pilot1.sch (EAGLE design)
At the start: 36 parts, among them SW1 SPST_TACT-KMR2, T1 SO8, T2 SO8, U1 MC-33926, U2 MC-33926

Commit message: .
Connections:
- net GND: no longer R5.2, R6.2
- net M2_A: now also JP2.4; no longer JP1.2
- net M2_B: now also JP1.2; no longer JP2.4
- net M2_POWER+: now also U2.OUT2, U2.OUT2_2, U2.OUT2_3, U2.OUT2_4; no longer U2.OUT1, U2.OUT1_2, U2.OUT1_3, U2.OUT1_4
- net M2_POWER-: now also U2.OUT1, U2.OUT1_2, U2.OUT1_3, U2.OUT1_4; no longer U2.OUT2, U2.OUT2_2, U2.OUT2_3, U2.OUT2_4
- net VDD: now also R5.2, R6.2
Other:
- note added: "FB needs components"
- note added: "IRF7342PBF"
- note added: "gyro needs to be completed"
- note added: "only need one protection circuit"
Changed lines of the file:
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@@
 <sheet>
 <plain>
+<text x="91.44" y="15.24" size="1.778" layer="91">IRF7342PBF </text>
+<text x="7.62" y="111.76" size="1.778" layer="91">FB needs components</text>
+<text x="93.98" y="203.2" size="1.778" layer="91">only need one protection circuit</text>
+<text x="215.9" y="83.82" size="1.778" layer="91">gyro needs to be completed</text>
 </plain>
 <instances>
@@
 </segment>
 <segment>
-<wire x1="83.82" y1="152.4" x2="91.44" y2="152.4" width="0.1524" layer="91"/>
-<label x="86.36" y="152.4" size="1.778" layer="95"/>
-<pinref part="R6" gate="G$1" pin="2"/>
-</segment>
-<segment>
 <wire x1="78.74" y1="162.56" x2="83.82" y2="162.56" width="0.1524" layer="91"/>
 <label x="78.74" y="162.56" size="1.778" layer="95"/>
@@
 <label x="78.74" y="68.58" size="1.778" layer="95"/>
 <pinref part="R12" gate="G$1" pin="2"/>
-</segment>
-<segment>
-<wire x1="78.74" y1="58.42" x2="83.82" y2="58.42" width="0.1524" layer="91"/>
-<label x="78.74" y="58.42" size="1.778" layer="95"/>
-<pinref part="R5" gate="G$1" pin="2"/>
 </segment>
 <segment>
@@
 </segment>
 <segment>
+<pinref part="U2" gate="A" pin="OUT2"/>
+<wire x1="15.24" y1="63.5" x2="30.48" y2="63.5" width="0.1524" layer="91"/>
+<pinref part="U2" gate="A" pin="OUT2_2"/>
+<wire x1="30.48" y1="63.5" x2="35.56" y2="63.5" width="0.1524" layer="91"/>
+<wire x1="35.56" y1="55.88" x2="30.48" y2="55.88" width="0.1524" layer="91"/>
+<wire x1="30.48" y1="55.88" x2="30.48" y2="58.42" width="0.1524" layer="91"/>
+<junction x="30.48" y="63.5"/>
+<pinref part="U2" gate="A" pin="OUT2_3"/>
+<wire x1="30.48" y1="58.42" x2="30.48" y2="60.96" width="0.1524" layer="91"/>
+<wire x1="30.48" y1="60.96" x2="30.48" y2="63.5" width="0.1524" layer="91"/>
+<wire x1="35.56" y1="58.42" x2="30.48" y2="58.42" width="0.1524" layer="91"/>
+<junction x="30.48" y="58.42"/>
+<pinref part="U2" gate="A" pin="OUT2_4"/>
+<wire x1="35.56" y1="60.96" x2="30.48" y2="60.96" width="0.1524" layer="91"/>
+<junction x="30.48" y="60.96"/>
+<label x="12.7" y="63.5" size="1.778" layer="95"/>
+</segment>
+</net>
+<net name="M2_POWER-" class="2">
+<segment>
+<pinref part="M2" gate="A" pin="5"/>
+<wire x1="116.84" y1="86.36" x2="96.52" y2="86.36" width="0.1524" layer="91"/>
+<label x="93.98" y="86.36" size="1.778" layer="95"/>
+</segment>
+<segment>
 <pinref part="U2" gate="A" pin="OUT1"/>
 <wire x1="15.24" y1="50.8" x2="30.48" y2="50.8" width="0.1524" layer="91"/>
@@
 </segment>
 </net>
-<net name="M2_POWER-" class="2">
-<segment>
-<pinref part="M2" gate="A" pin="5"/>
-<wire x1="116.84" y1="86.36" x2="96.52" y2="86.36" width="0.1524" layer="91"/>
-<label x="93.98" y="86.36" size="1.778" layer="95"/>
-</segment>
-<segment>
-<pinref part="U2" gate="A" pin="OUT2"/>
-<wire x1="15.24" y1="63.5" x2="30.48" y2="63.5" width="0.1524" layer="91"/>
-<pinref part="U2" gate="A" pin="OUT2_2"/>
-<wire x1="30.48" y1="63.5" x2="35.56" y2="63.5" width="0.1524" layer="91"/>
-<wire x1="35.56" y1="55.88" x2="30.48" y2="55.88" width="0.1524" layer="91"/>
-<wire x1="30.48" y1="55.88" x2="30.48" y2="58.42" width="0.1524" layer="91"/>
-<junction x="30.48" y="63.5"/>
-<pinref part="U2" gate="A" pin="OUT2_3"/>
-<wire x1="30.48" y1="58.42" x2="30.48" y2="60.96" width="0.1524" layer="91"/>
-<wire x1="30.48" y1="60.96" x2="30.48" y2="63.5" width="0.1524" layer="91"/>
-<wire x1="35.56" y1="58.42" x2="30.48" y2="58.42" width="0.1524" layer="91"/>
-<junction x="30.48" y="58.42"/>
-<pinref part="U2" gate="A" pin="OUT2_4"/>
-<wire x1="35.56" y1="60.96" x2="30.48" y2="60.96" width="0.1524" layer="91"/>
-<junction x="30.48" y="60.96"/>
-<label x="12.7" y="63.5" size="1.778" layer="95"/>
-</segment>
-</net>
 <net name="VDD" class="1">
 <segment>
@@
 <pinref part="R10" gate="G$1" pin="2"/>
 </segment>
+<segment>
+<wire x1="83.82" y1="152.4" x2="91.44" y2="152.4" width="0.1524" layer="91"/>
+<label x="86.36" y="152.4" size="1.778" layer="95"/>
+<pinref part="R6" gate="G$1" pin="2"/>
+</segment>
+<segment>
+<wire x1="78.74" y1="58.42" x2="83.82" y2="58.42" width="0.1524" layer="91"/>
+<label x="78.74" y="58.42" size="1.778" layer="95"/>
+<pinref part="R5" gate="G$1" pin="2"/>
+</segment>
 </net>
 <net name="M1_B" class="0">
@@
 <net name="M2_B" class="0">
 <segment>
+<wire x1="116.84" y1="93.98" x2="96.52" y2="93.98" width="0.1524" layer="91"/>
+<label x="93.98" y="93.98" size="1.778" layer="95"/>
+<pinref part="M2" gate="A" pin="2"/>
+</segment>
+<segment>
+<pinref part="JP1" gate="A" pin="2"/>
+<wire x1="208.28" y1="187.96" x2="208.28" y2="195.58" width="0.1524" layer="91"/>
+<label x="208.28" y="193.04" size="1.778" layer="95" rot="R90"/>
+</segment>
+</net>
+<net name="M2_A" class="0">
+<segment>
+<wire x1="116.84" y1="91.44" x2="96.52" y2="91.44" width="0.1524" layer="91"/>
+<label x="93.98" y="91.44" size="1.778" layer="95"/>
+<pinref part="M2" gate="A" pin="3"/>
+</segment>
+<segment>
 <pinref part="JP2" gate="A" pin="4"/>
 <wire x1="228.6" y1="187.96" x2="228.6" y2="195.58" width="0.1524" layer="91"/>
 <label x="228.6" y="193.04" size="1.778" layer="95" rot="R90"/>
 </segment>
-<segment>
-<wire x1="116.84" y1="93.98" x2="96.52" y2="93.98" width="0.1524" layer="91"/>
-<label x="93.98" y="93.98" size="1.778" layer="95"/>
-<pinref part="M2" gate="A" pin="2"/>
-</segment>
-</net>
-<net name="M2_A" class="0">
-<segment>
-<wire x1="116.84" y1="91.44" x2="96.52" y2="91.44" width="0.1524" layer="91"/>
-<label x="93.98" y="91.44" size="1.778" layer="95"/>
-<pinref part="M2" gate="A" pin="3"/>
-</segment>
-<segment>
-<pinref part="JP1" gate="A" pin="2"/>
-<wire x1="208.28" y1="187.96" x2="208.28" y2="195.58" width="0.1524" layer="91"/>
-<label x="208.28" y="193.04" size="1.778" layer="95" rot="R90"/>
-</segment>
-</net>
+</net>

Commit message: .
Parts:
- removed D1, D2: 12V, diode:ZENER-DIODESOT23
- removed R1: 100k, Triple_Axis_Accelerometer-Gyro_Breakout_-_MPU-6050_v12:RESISTOR0805-RES
- removed SW1: SPST_TACT-KMR2, adafruit:SPST_TACT-KMR2
- removed T1, T2: SO8, zetex:NMOS2SO8
- removed U$1: MPU-6050-1, Triple_Axis_Accelerometer-Gyro_Breakout_-_MPU-6050_v12:MPU-6050-1
- added BUMPR: (no value), pinhead:PINHD-1X3/90
- added C10: .1uf, SparkFun-Passives:CAP0805
- added C11, C13: .47uf, Triple_Axis_Accelerometer-Gyro_Breakout_-_MPU-6050_v12:CAP0805
- added C8: 10nf, SparkFun-Passives:CAP0805
- added C9: 2.2nf, SparkFun-Passives:CAP0805
- added ESC_ENA: RED, SparkFun-LED:LED-RED0603
- added HEARTBEAT: BLUE, SparkFun-LED:LED-BLUE0603
- added JP_ENA: (no value), pinhead:PINHD-1X2
- added M1_AUX, M2_AUX: (no value), pinhead:PINHD-1X2/90
- added POWER: GREEN, SparkFun-LED:LED-GREEN0603
- added R14, R15: 220, Triple_Axis_Accelerometer-Gyro_Breakout_-_MPU-6050_v12:RESISTOR0805-RES
- added R16, R17, R20, R21, R22: 1k, Triple_Axis_Accelerometer-Gyro_Breakout_-_MPU-6050_v12:RESISTOR0805-RES
- added R18, R19, R2: 10k, Triple_Axis_Accelerometer-Gyro_Breakout_-_MPU-6050_v12:RESISTOR0805-RES
- added RESET: SPST_TACT-KMR2, adafruit:SPST_TACT-KMR2
- added U3: MPU-6050-1, Triple_Axis_Accelerometer-Gyro_Breakout_-_MPU-6050_v12:MPU-6050-1
- added UTIL: (no value), pinhead:PINHD-1X4/90
- M1, M2: device pinhead:PINHD-1X6 -> pinhead:PINHD-1X6/90
- MOTOR_POWER_IN: value (none) -> 1X2-3.5MM; device pinhead:PINHD-1X2 -> adafruit:1X2-3.5MM
- R13: value 100k -> 10k
Connections:
- net PWM1 renamed M1_PWM
- net PWM2 renamed M2_PWM
- removed net N$13: D2.C, R1.2, T2A.G
- removed net N$14: D1.C, R13.2, T1A.G
- new net ESC_EN_JP: JP1.5, JP_ENA.1
- new net HB: HEARTBEAT.A, JP1.6
- new net N$17: C9.1, U3.CPOUT
- new net N$18: C10.1, U3.REGOUT
- new net N$19: C8.1, U3.VLOGIC
- new net N$20: R14.1, R16.1, U2.FB
- new net N$21: POWER.C, R20.2
- new net N$22: R15.1, R17.1, U1.FB
- new net N$23: ESC_ENA.C, R21.2
- new net N$24: HEARTBEAT.C, R22.2
- new net S1: BUMPR.3, JP2.5
- new net S2: JP1.3, UTIL.3
- new net S3: JP4.3, UTIL.4
- net 3V3: now also R13.1, R2.1, U3.VDD; no longer U$1.VDD
- net AUX_SCL: now also U3.AUX_CL; no longer U$1.AUX_CL
- net AUX_SDA: now also U3.AUX_DA; no longer U$1.AUX_DA
- net ESC_EN: now also ESC_ENA.A, JP_ENA.2; no longer JP1.5
- net GND: now also BUMPR.1, C10.2, C11.1, C13.1, C8.2, C9.2, M1.4, M2.4, R14.2, R15.2, R20.1, R21.1, R22.1, RESET.S, RESET.S1, U3.AD0, U3.CLKIN, U3.FSYNC, U3.GND, UTIL.1; no longer D1.A, D2.A, M1.1, M2.1, SW1.S, SW1.S1, T1A.D, T1A.S, T2A.D, T2A.S, U$1.GND
- net IMU_INT: now also U3.INT; no longer U$1.INT
- net M1_A: now also M1.5; no longer M1.3
- net M1_B: now also M1.6; no longer M1.2
- net M1_FB: now also C13.2, R17.2; no longer U1.FB
- net M1_POWER+: now also M1.2, M1_AUX.2; no longer M1.6
- net M1_POWER-: now also M1.1, M1_AUX.1; no longer M1.5
- net M2_A: now also M2.5; no longer M2.3
- net M2_B: now also M2.6; no longer M2.2
- net M2_DIR: now also JP4.4; no longer JP1.3
- net M2_FB: now also C11.2, R16.2; no longer U2.FB
- net M2_POWER+: now also M2.2, M2_AUX.2; no longer M2.6
- net M2_POWER-: now also M2.1, M2_AUX.1; no longer M2.5
- net N$15: now also R18.2
- net N$16: now also R19.2
- net RESET: now also RESET.P, RESET.P1; no longer SW1.P, SW1.P1
- net SCL: now also R13.2, U3.SCL; no longer U$1.SCL
- net SDA: now also R2.2, U3.SDA; no longer U$1.SDA
- net VDD: now also BUMPR.2, M1.3, M2.3, POWER.A, R18.1, R19.1, UTIL.2; no longer M1.4, M2.4
- net VPWR: no longer R1.1, R13.1
Other:
- note removed: "FB needs components"
- note removed: "IRF7342PBF"
- note removed: "gyro needs to be completed"
- note removed: "only need one protection circuit"
- moved on the sheet: AUX_I2C, C1, C4, C5, C6, C7, M1, M2, R10, R11, R12, R13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

Commit message: .
Parts:
- removed AUX_I2C: (no value), pinhead:PINHD-1X4
- removed R22: 1k, Triple_Axis_Accelerometer-Gyro_Breakout_-_MPU-6050_v12:RESISTOR0805-RES
- added C12: .1uf, Triple_Axis_Accelerometer-Gyro_Breakout_-_MPU-6050_v12:CAP0805
- added R1: 1k, Triple_Axis_Accelerometer-Gyro_Breakout_-_MPU-6050_v12:RESISTOR0805-RES
- C1: value 47uf -> .1uf; device SparkFun-Capacitors:47UF-50V-20%(ELECT) -> Triple_Axis_Accelerometer-Gyro_Breakout_-_MPU-6050_v12:CAP0805
- C10: value .1uf -> 1uf; device SparkFun-Passives:CAP0805 -> Triple_Axis_Accelerometer-Gyro_Breakout_-_MPU-6050_v12:CAP0805
- C11: value .47uf -> 47uf; device Triple_Axis_Accelerometer-Gyro_Breakout_-_MPU-6050_v12:CAP0805 -> SparkFun-Capacitors:47UF-50V-20%(ELECT)
- C13: value .47uf -> 1uf
- C2: value 47uf -> 33nf; device SparkFun-Capacitors:47UF-50V-20%(ELECT) -> Triple_Axis_Accelerometer-Gyro_Breakout_-_MPU-6050_v12:CAP0805
- C3: value 47uf -> 2.2nf; device SparkFun-Capacitors:47UF-50V-20%(ELECT) -> SparkFun-Passives:CAP0805
- C4: value 33nf -> 47uf; device Triple_Axis_Accelerometer-Gyro_Breakout_-_MPU-6050_v12:CAP0805 -> SparkFun-Capacitors:47UF-50V-20%(ELECT)
- C6: value 47uf -> 10nf; device SparkFun-Capacitors:47UF-50V-20%(ELECT) -> SparkFun-Passives:CAP0805
- C7: device Triple_Axis_Accelerometer-Gyro_Breakout_-_MPU-6050_v12:CAP0805 -> SparkFun-Passives:CAP0805
- C8: value 10nf -> .47uf; device SparkFun-Passives:CAP0805 -> Triple_Axis_Accelerometer-Gyro_Breakout_-_MPU-6050_v12:CAP0805
- C9: value 2.2nf -> .47uf; device SparkFun-Passives:CAP0805 -> Triple_Axis_Accelerometer-Gyro_Breakout_-_MPU-6050_v12:CAP0805
- PCB1: value ARDUINO_UNO -> ARDUINO_UNO_EXT; device E14_Arduino_published:ARDUINO_UNO -> E14_Arduino_published:ARDUINO_UNO_EXT
- R11, R12, R20, R9: value 1k -> 10k
- R13, R18: value 10k -> 1k
- R14, R15: value 220 -> 1k
- R19, R2: value 10k -> 220
- U2: value MC-33926 -> MPU-6050-1; device Freescale-MC33926PNB:FREESCALE-MC33926PNB -> Triple_Axis_Accelerometer-Gyro_Breakout_-_MPU-6050_v12:MPU-6050-1
- U3: value MPU-6050-1 -> MC-33926; device Triple_Axis_Accelerometer-Gyro_Breakout_-_MPU-6050_v12:MPU-6050-1 -> Freescale-MC33926PNB:FREESCALE-MC33926PNB
Connections:
- removed net AUX_SCL: AUX_I2C.4, U3.AUX_CL
- removed net AUX_SDA: AUX_I2C.3, U3.AUX_DA
- new net AGND: U1.AGND, U1.AGND_2
- new net PGND: C1.2, C10.2, C11.-, C12.2, C13.2, C4.-, MOTOR_POWER_IN.1, U1.PGND, U1.PGND_2, U1.PGND_3, U1.PGND_4, U1.PGND_5, U1.PGND_6, U3.PGND, U3.PGND_2, U3.PGND_3, U3.PGND_4, U3.PGND_5, U3.PGND_6
- net 3V3: now also R11.1, R9.1, U2.VDD; no longer AUX_I2C.2, R13.1, R2.1, U3.VDD
- net ESC_EN: now also R17.2, R7.2; no longer R3.2, R4.2
- net GND: now also C3.2, C6.2, C8.1, C9.1, R1.2, R10.2, R13.2, R19.2, R2.2, R21.2, R4.1, R6.1, R8.1, U2.AD0, U2.CLKIN, U2.FSYNC, U2.GND, U3.AGND, U3.AGND_2; no longer AUX_I2C.1, C1.-, C10.2, C11.1, C13.1, C2.-, C3.-, C6.-, C8.2, C9.2, MOTOR_POWER_IN.1, R11.2, R12.2, R14.2, R15.2, R20.1, R21.1, R22.1, R8.2, R9.2, U1.AGND, U1.AGND_2, U1.NC, U1.NC_2, U1.NC_3, U1.PGND, U1.PGND_2, U1.PGND_3, U1.PGND_4, U1.PGND_5, U1.PGND_6, U2.AGND, U2.AGND_2, U2.NC, U2.NC_2, U2.NC_3, U2.PGND, U2.PGND_2, U2.PGND_3, U2.PGND_4, U2.PGND_5, U2.PGND_6, U3.AD0, U3.CLKIN, U3.FSYNC, U3.GND
- net IMU_INT: now also U2.INT; no longer U3.INT
- net M1_A: now also M2.5; no longer M1.5
- net M1_B: now also M2.6; no longer M1.6
- net M1_DIR: now also U3.INV; no longer U1.INV
- net M1_FB: now also C8.2, R14.2; no longer C13.2, R17.2
- net M1_POWER+: now also M2.2, U3.OUT2, U3.OUT2_2, U3.OUT2_3, U3.OUT2_4; no longer M1.2, U1.OUT2, U1.OUT2_2, U1.OUT2_3, U1.OUT2_4
- net M1_POWER-: now also M2.1, U3.OUT1, U3.OUT1_2, U3.OUT1_3, U3.OUT1_4; no longer M1.1, U1.OUT1, U1.OUT1_2, U1.OUT1_3, U1.OUT1_4
- net M1_PWM: now also U3.!D2; no longer U1.!D2
- net M2_A: now also M1.5; no longer M2.5
- net M2_B: now also M1.6; no longer M2.6
- net M2_DIR: now also U1.INV; no longer U2.INV
- net M2_FB: now also C9.2, R18.2; no longer C11.2, R16.2
- net M2_POWER+: now also M1.2, U1.OUT2, U1.OUT2_2, U1.OUT2_3, U1.OUT2_4; no longer M2.2, U2.OUT2, U2.OUT2_2, U2.OUT2_3, U2.OUT2_4
- net M2_POWER-: now also M1.1, U1.OUT1, U1.OUT1_2, U1.OUT1_3, U1.OUT1_4; no longer M2.1, U2.OUT1, U2.OUT1_2, U2.OUT1_3, U2.OUT1_4
- net M2_PWM: now also U1.!D2; no longer U2.!D2
- net N$1: now also R17.1, U3.EN; no longer R3.1, U1.EN
- net N$10: now also R16.1, U3.IN2; no longer R7.1, U1.IN2
- net N$11: now also R21.1, U3.D1; no longer R8.1, U1.D1
- net N$12: now also R13.1, U3.IN1; no longer R9.1, U1.IN1
- net N$15: now also R12.2, U1.!SF; no longer R18.2, U2.!SF
- net N$16: now also R20.2, U3.!SF; no longer R19.2, U1.!SF
- net N$17: now also C3.1, U2.CPOUT; no longer C9.1, U3.CPOUT
- net N$18: now also C7.1, U2.REGOUT; no longer C10.1, U3.REGOUT
- net N$19: now also C6.1, U2.VLOGIC; no longer C8.1, U3.VLOGIC
- net N$2: now also R10.1, U1.D1; no longer R12.1, U2.D1
- net N$20: now also R18.1, R2.1, U1.FB; no longer R14.1, R16.1, U2.FB
- net N$21: now also R4.2; no longer R20.2
- net N$22: now also R14.1, R19.1, U3.FB; no longer R15.1, R17.1, U1.FB
- net N$23: now also R8.2; no longer R21.2
- net N$24: now also R6.2; no longer R22.2
- net N$3: now also R3.1, U1.SLEW; no longer R5.1, U2.SLEW
- net N$4: now also R15.1, U3.SLEW; no longer R6.1, U1.SLEW
- net N$5: now also C5.1, U3.CCP; no longer C4.1, U1.CCP
- net N$6: now also C2.1, U1.CCP; no longer C5.1, U2.CCP
- net N$7: now also R7.1, U1.EN; no longer R4.1, U2.EN
- net N$8: now also R5.1, U1.IN2; no longer R10.1, U2.IN2
- net N$9: now also R1.1, U1.IN1; no longer R11.1, U2.IN1
- net SCL: now also R9.2, U2.SCL; no longer R13.2, U3.SCL
- net SDA: now also R11.2, U2.SDA; no longer R2.2, U3.SDA
- net VDD: now also R12.1, R15.2, R16.2, R20.1, R3.2; no longer R10.2, R18.1, R19.1, R6.2, R7.2
- net VPWR: now also C1.1, C10.1, C11.+, C12.1, C13.1, C2.2, C4.+, U3.VPWR, U3.VPWR_2, U3.VPWR_3, U3.VPWR_4; no longer C1.+, C2.+, C3.+, C4.2, C6.+, C7.1, U2.VPWR, U2.VPWR_2, U2.VPWR_3, U2.VPWR_4
Other:
- moved on the sheet: C10, C13, C5, C7, C8, C9, M1, M1_AUX, M2, M2_AUX, R10, R11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

Commit message: .
Connections:
- net M1_A: now also M1.5; no longer M2.5
- net M1_B: now also M1.6; no longer M2.6
- net M1_POWER+: now also M1.2; no longer M2.2
- net M1_POWER-: now also M1.1; no longer M2.1
- net M2_A: now also M2.5; no longer M1.5
- net M2_B: now also M2.6; no longer M1.6
- net M2_POWER+: now also M2.2; no longer M1.2
- net M2_POWER-: now also M2.1; no longer M1.1
Other:
- moved on the sheet: M1, M2
Changed lines of the file:
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@@
 <part name="MOTOR_POWER_IN" library="adafruit" deviceset="1X2" device="-3.5MM"/>
 <part name="U2" library="Triple_Axis_Accelerometer-Gyro_Breakout_-_MPU-6050_v12" deviceset="MPU-6050" device="-1"/>
+<part name="M1" library="pinhead" deviceset="PINHD-1X6" device="/90"/>
 <part name="M2" library="pinhead" deviceset="PINHD-1X6" device="/90"/>
-<part name="M1" library="pinhead" deviceset="PINHD-1X6" device="/90"/>
 <part name="C5" library="Triple_Axis_Accelerometer-Gyro_Breakout_-_MPU-6050_v12" deviceset="CAP" device="0805" value="33nf"/>
 <part name="C2" library="Triple_Axis_Accelerometer-Gyro_Breakout_-_MPU-6050_v12" deviceset="CAP" device="0805" value="33nf"/>
@@
 <instance part="MOTOR_POWER_IN" gate="G$1" x="137.16" y="127"/>
 <instance part="U2" gate="G$1" x="213.36" y="93.98"/>
-<instance part="M2" gate="A" x="137.16" y="106.68"/>
-<instance part="M1" gate="A" x="137.16" y="68.58"/>
+<instance part="M1" gate="A" x="137.16" y="106.68"/>
+<instance part="M2" gate="A" x="137.16" y="68.58"/>
 <instance part="C5" gate="G$1" x="33.02" y="124.46" rot="R270"/>
 <instance part="C2" gate="G$1" x="30.48" y="33.02" rot="R270"/>
@@
 <segment>
 <wire x1="134.62" y1="106.68" x2="111.76" y2="106.68" width="0.1524" layer="91"/>
+<pinref part="M1" gate="A" pin="4"/>
+<pinref part="GND7" gate="1" pin="GND"/>
+</segment>
+<segment>
+<wire x1="134.62" y1="68.58" x2="111.76" y2="68.58" width="0.1524" layer="91"/>
 <pinref part="M2" gate="A" pin="4"/>
-<pinref part="GND7" gate="1" pin="GND"/>
-</segment>
-<segment>
-<wire x1="134.62" y1="68.58" x2="111.76" y2="68.58" width="0.1524" layer="91"/>
-<pinref part="M1" gate="A" pin="4"/>
 <pinref part="GND6" gate="1" pin="GND"/>
 </segment>
@@
 <wire x1="134.62" y1="111.76" x2="114.3" y2="111.76" width="0.1524" layer="91"/>
 <label x="111.76" y="111.76" size="1.778" layer="95"/>
-<pinref part="M2" gate="A" pin="2"/>
+<pinref part="M1" gate="A" pin="2"/>
 </segment>
 <segment>
@@
 <label x="111.76" y="114.3" size="1.778" layer="95"/>
 <wire x1="134.62" y1="114.3" x2="114.3" y2="114.3" width="0.1524" layer="91"/>
-<pinref part="M2" gate="A" pin="1"/>
+<pinref part="M1" gate="A" pin="1"/>
 </segment>
 <segment>
@@
 <wire x1="134.62" y1="73.66" x2="114.3" y2="73.66" width="0.1524" layer="91"/>
 <label x="111.76" y="73.66" size="1.778" layer="95"/>
-<pinref part="M1" gate="A" pin="2"/>
+<pinref part="M2" gate="A" pin="2"/>
 </segment>
 <segment>
@@
 <label x="111.76" y="76.2" size="1.778" layer="95"/>
 <wire x1="134.62" y1="76.2" x2="114.3" y2="76.2" width="0.1524" layer="91"/>
-<pinref part="M1" gate="A" pin="1"/>
+<pinref part="M2" gate="A" pin="1"/>
 </segment>
 <segment>
@@
 <wire x1="134.62" y1="109.22" x2="114.3" y2="109.22" width="0.1524" layer="91"/>
 <label x="111.76" y="109.22" size="1.778" layer="95"/>
-<pinref part="M2" gate="A" pin="3"/>
+<pinref part="M1" gate="A" pin="3"/>
 </segment>
 <segment>
 <wire x1="134.62" y1="71.12" x2="114.3" y2="71.12" width="0.1524" layer="91"/>
 <label x="111.76" y="71.12" size="1.778" layer="95"/>
-<pinref part="M1" gate="A" pin="3"/>
+<pinref part="M2" gate="A" pin="3"/>
 </segment>
 <segment>
@@
 </segment>
 <segment>
-<pinref part="M2" gate="A" pin="6"/>
+<pinref part="M1" gate="A" pin="6"/>
 <wire x1="134.62" y1="101.6" x2="114.3" y2="101.6" width="0.1524" layer="91"/>
 <label x="111.76" y="101.6" size="1.778" layer="95"/>
@@
 </segment>
 <segment>
-<pinref part="M2" gate="A" pin="5"/>
+<pinref part="M1" gate="A" pin="5"/>
 <wire x1="134.62" y1="104.14" x2="114.3" y2="104.14" width="0.1524" layer="91"/>
 <label x="111.76" y="104.14" size="1.778" layer="95"/>
@@
 </segment>
 <segment>
-<pinref part="M1" gate="A" pin="6"/>
+<pinref part="M2" gate="A" pin="6"/>
 <wire x1="134.62" y1="63.5" x2="114.3" y2="63.5" width="0.1524" layer="91"/>
 <label x="111.76" y="63.5" size="1.778" layer="95"/>
@@
 </segment>
 <segment>
-<pinref part="M1" gate="A" pin="5"/>
+<pinref part="M2" gate="A" pin="5"/>
 <wire x1="134.62" y1="66.04" x2="114.3" y2="66.04" width="0.1524" layer="91"/>
 <label x="111.76" y="66.04" size="1.778" layer="95"/>
