File: Eagle/s3-pilot2.brd (EAGLE design)
At the start: 57.1 x 53.6 mm, 17 parts, among them J1 ARDUINO_R3_SHIELD, M2_1 ENA_JMP

Commit message: work session with David verified ESC work - problem was buttons on breadboard verify a few updates and eagle, then re-order Code needs to be split / merged / something to deal with various situations need 2-way serial now, since cant really use breadboard buttons anymore.
Connections:
- net M1_FB: now also J1.A2; no longer J1.A0
Changed lines of the file:
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@@
 </signal>
 <signal name="M1_FB">
-<contactref element="J1" pad="A0"/>
 <contactref element="U$1" pad="FB"/>
-<wire x1="20.32" y1="25.4" x2="41.91" y2="7.62" width="0" layer="19" extent="1-1"/>
+<contactref element="J1" pad="A2"/>
+<wire x1="20.32" y1="25.4" x2="46.99" y2="7.62" width="0" layer="19" extent="1-1"/>
 </signal>
 <signal name="N$3">
