File: Eagle/s3-pilot2.brd (EAGLE design)
At the start: 57.1 x 53.6 mm, 17 parts, among them J1 ARDUINO_R3_SHIELD, M2_1 ENA_JMP

Commit message: chkpt before changing ISR around - it is not working well - too fast?
Connections:
- new net 3.3: J1.3.3V, MPU6050.VCC
- net GND: now also J1.GND@0, J1.GND@1
- net VDD: no longer MPU6050.VCC
Routing:
- net GND: track 151.5 -> 0.00 mm
- net VDD: track 122.8 -> 0.00 mm
- net M1_A: track 78.4 -> 0.00 mm
- net PWM_X: track 69.9 -> 0.00 mm
- net M1_B: track 69.6 -> 0.00 mm
- net ESC_EN: track 54.3 -> 0.00 mm
- net M2_FB: track 52.3 -> 0.00 mm
- net RESET: track 52.2 -> 0.00 mm
- net N$3: track 51.1 -> 0.00 mm, vias 1 -> 0
- net M1_PWM: track 48.8 -> 0.00 mm, vias 1 -> 0
- net M2_A: track 46.2 -> 0.00 mm
- net M2_DIR: track 45.8 -> 0.00 mm
- net IMU_INT: track 42.3 -> 0.00 mm
- net N$21: track 37.6 -> 0.00 mm
- net ESC_EN_JMP: track 35.8 -> 0.00 mm
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
Commit message: working basically, still need to correct x/y/h stuff (as usual) added remote reset jumper for arduino to sch
Parts:
- added JP1: Reset, pinhead:1X02/90
- moved R1 38.1 mm to (44.5, 48.3)
Connections:
- net GND: now also JP1.1
- net RESET: now also JP1.2
Changed lines of the file:
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@@
 <param name="TopRouterVariant" value="1"/>
 <param name="tpViaShape" value="round"/>
-<param name="PrefDir.1" value="a"/>
+<param name="PrefDir.1" value="*"/>
 <param name="PrefDir.2" value="0"/>
 <param name="PrefDir.3" value="0"/>
@@
 <param name="PrefDir.14" value="0"/>
 <param name="PrefDir.15" value="0"/>
-<param name="PrefDir.16" value="a"/>
+<param name="PrefDir.16" value="-"/>
 <param name="cfVia" value="8"/>
 <param name="cfNonPref" value="5"/>
@@
 <attribute name="PROD_ID" value="DIO-00862" x="15.24" y="31.75" size="1.778" layer="27" rot="R270" display="off"/>
 </element>
-<element name="R1" library="SparkFun-Passives" package="1206" value="1k" x="10.16" y="31.75" rot="R270"/>
+<element name="R1" library="SparkFun-Passives" package="1206" value="1k" x="44.45" y="48.26" rot="R270"/>
 <element name="R4" library="SparkFun-Passives" package="1206" value="1k" x="40.64" y="31.75" rot="R270"/>
 <element name="R6" library="SparkFun-Passives" package="1206" value="1k" x="30.48" y="31.75" rot="R90"/>
@@
 <attribute name="VALUE" x="50.8" y="43.815" size="1.27" layer="27"/>
 </element>
+<element name="JP1" library="pinhead" package="1X02/90" value="Reset" x="13.97" y="7.62" rot="R180"/>
 </elements>
 <signals>
@@
 <contactref element="J1" pad="GND@0"/>
 <contactref element="J1" pad="GND@1"/>
+<contactref element="JP1" pad="1"/>
 </signal>
 <signal name="VDD" class="1">
@@
 <contactref element="U$3" pad="IN2"/>
 <contactref element="U$1" pad="IN2"/>
-<wire x1="35.56" y1="25.4" x2="50.8" y2="17.78" width="0" layer="19" extent="1-1"/>
+<wire x1="35.56" y1="25.4" x2="44.45" y2="49.66" width="0" layer="19" extent="1-1"/>
 <wire x1="33.02" y1="25.4" x2="35.56" y2="25.4" width="0" layer="19" extent="1-1"/>
+<wire x1="50.8" y1="17.78" x2="35.56" y2="25.4" width="0" layer="19" extent="1-1"/>
 <wire x1="20.32" y1="38.1" x2="33.02" y2="25.4" width="0" layer="19" extent="1-1"/>
 <wire x1="17.78" y1="38.1" x2="20.32" y2="38.1" width="0" layer="19" extent="1-1"/>
 <wire x1="15.24" y1="33.25" x2="17.78" y2="38.1" width="0" layer="19" extent="1-1"/>
-<wire x1="10.16" y1="33.15" x2="15.24" y2="33.25" width="0" layer="19" extent="1-1"/>
-<wire x1="5.08" y1="45.72" x2="10.16" y2="33.15" width="0" layer="19" extent="1-1"/>
+<wire x1="5.08" y1="45.72" x2="17.78" y2="38.1" width="0" layer="19" extent="1-1"/>
 <wire x1="29.21" y1="7.62" x2="33.02" y2="25.4" width="0" layer="19" extent="1-1"/>
-<wire x1="5.08" y1="10.16" x2="10.16" y2="33.15" width="0" layer="19" extent="1-1"/>
+<wire x1="5.08" y1="10.16" x2="29.21" y2="7.62" width="0" layer="19" extent="1-1"/>
 </signal>
 <signal name="M1_B">
@@
 <contactref element="S1" pad="3"/>
 <contactref element="S1" pad="4"/>
+<contactref element="JP1" pad="2"/>
 <wire x1="50.165" y1="28.956" x2="50.165" y2="34.544" width="0" layer="19" extent="1-1"/>
 <wire x1="24.13" y1="7.62" x2="50.165" y2="28.956" width="0" layer="19" extent="1-1"/>
+<wire x1="12.7" y1="11.43" x2="24.13" y2="7.62" width="0" layer="19" extent="1-1"/>
 </signal>
 <signal name="N$21">
@@
 <contactref element="R1" pad="2"/>
 <contactref element="JP5" pad="2"/>
-<wire x1="10.16" y1="30.35" x2="50.8" y2="46.99" width="0" layer="19" extent="1-1"/>
+<wire x1="44.45" y1="46.86" x2="50.8" y2="46.99" width="0" layer="19" extent="1-1"/>
 </signal>
 <signal name="3.3">

Commit message: eagle updates - brd not complete
Parts:
- removed S1: RESET, SparkFun-Electromechanical:TACTILE-SWITCH-SMD
- added RESET: RESET, SparkFun-Electromechanical:TACTILE_SWITCH_TALL
- JP1: device pinhead:1X02/90 -> pinhead:1X02
- M2_1: value ENA_JMP -> ENA
- U$1: value MC33926-SINGLE-BO -> M1
- moved JP1 51.4 mm to (53.3, 40.6), turned to 270 degrees
- renumbered ESC_ENA to ENABLE, J1 to GND
Connections:
- removed net N$1: GND.SCL, MPU6050.SCL
- removed net N$2: GND.SDA, MPU6050.SDA
- new net SCL: GND.A5, GND.SCL, MPU6050.SCL
- new net SDA: GND.A4, GND.SDA, MPU6050.SDA
- net GND: now also RESET.A2; no longer S1.1, S1.2
- net M1_FB: now also GND.A2; no longer GND.A0
- net RESET: now also RESET.B2; no longer S1.3, S1.4
Routing:
- added copper zone on layer 1, net N$1
- removed copper zone on layer 1, net GND
Other:
- board text added: "GND"
- board text added: "S3-PILOT2 3/28/15"
- board text removed: "S3-PILOT 2/27/15"
